Commit message: Finshed OAK Onboard inference.

File: depthai-ros/depthai_bridge/urdf/sentry_descr.urdf.xacro (robot description, xacro)
@@ -41,4 +41,10 @@
         <limit effort="30" velocity="10.0" lower="-3.14" upper="3.14" />
     </joint>
+    <link name="daheng_img_frame"/>
+    <joint name="daheng_joint" type="fixed">
+        <parent link="gimbal_pitch_frame"/>
+        <child link="daheng_img_frame"/>
+        <origin xyz="0.1 0 0.05" rpy="-1.57 0 -1.57" />
+    </joint>
     <joint name="$(arg camera_name)_center_joint" type="fixed">
         <parent link="gimbal_yaw_frame"/>

Commit message: Pre-Open Update(RMUL major changes added).

File: depthai-ros/depthai_bridge/urdf/sentry_descr.urdf.xacro (robot description, xacro)
@@ -25,9 +25,15 @@
     <!-- Yaw axis of robot -->
     <link name="gimbal_yaw_frame"/>
+    <joint name="base_joint" type="fixed">
+        <parent link="$(arg parent_frame)"/>
+        <child link="gimbal_yaw_frame"/>
+        <origin xyz="0 0 0" rpy="0 0 0" />
+    </joint>
+    <link name="chassis_frame"/>
     <joint name="gimbal_yaw_joint" type="revolute">
         <axis xyz="0 0 1"/>
-        <origin xyz="0 0 0.25" rpy="0 0 0" />
-        <parent link="$(arg parent_frame)"/>
-        <child link="gimbal_yaw_frame"/>
+        <origin xyz="0 0 -0.25" rpy="0 0 0" />
+        <parent link="gimbal_yaw_frame"/>
+        <child link="chassis_frame"/>
         <limit effort="30" velocity="10.0" lower="-3.14" upper="3.14" />
     </joint>
@@ -37,5 +43,5 @@
         <axis xyz="0 1 0"/>
         <origin xyz="0 0 0.25" rpy="0 0 0" />
-        <parent link="gimbal_yaw_frame"/>
+        <parent link="$(arg parent_frame)"/>
         <child link="gimbal_pitch_frame"/>
         <limit effort="30" velocity="10.0" lower="-3.14" upper="3.14" />
@@ -47,4 +53,16 @@
         <origin xyz="0.1 0 0.05" rpy="-1.57 0 -1.57" />
     </joint>
+    <link name="usb_left_frame"/>
+    <joint name="usb_left_joint" type="fixed">
+        <parent link="gimbal_yaw_frame"/>
+        <child link="usb_left_frame"/>
+        <origin xyz="0 0.1 0.15" rpy="-1.57 0 0" />
+    </joint>
+    <link name="usb_right_frame"/>
+    <joint name="usb_right_joint" type="fixed">
+        <parent link="gimbal_yaw_frame"/>
+        <child link="usb_right_frame"/>
+        <origin xyz="0 -0.1 0.15" rpy="1.57 3.14 0" />
+    </joint>
     <joint name="$(arg camera_name)_center_joint" type="fixed">
         <parent link="gimbal_yaw_frame"/>
