Commit message: Updated param.

File: LIO-SAM/config/robot.urdf.xacro (robot description, xacro)
@@ -13,5 +13,5 @@
     <parent link="base_link" />
     <child link="livox_frame" />
-    <origin xyz="0 0 0" rpy="3.14 0 0" />
+    <origin xyz="0 0 0.2" rpy="3.14 0 -1.57" />
   </joint>
   <link name="imu_link"> </link>

Commit message: Refined nav2 params.

File: LIO-SAM/config/robot.urdf.xacro (robot description, xacro)
@@ -13,5 +13,5 @@
     <parent link="base_link" />
     <child link="livox_frame" />
-    <origin xyz="0 0 0.2" rpy="3.14 0 -1.57" />
+    <origin xyz="0 0 0.0" rpy="3.14 0.0 -1.57" />
   </joint>
   <link name="imu_link"> </link>

Commit message: Deleted unnecessary files, fixed FASTLIO Support.

File: LIO-SAM/config/robot.urdf.xacro (robot description, xacro)
@@ -9,9 +9,33 @@
     <origin xyz="0 0 0" rpy="0 0 0" />
   </joint>
+  <link name="usb_left_frame"></link>
+  <joint name="usb_left_joint" type="fixed">
+    <parent link="base_link"/>
+    <child link="usb_left_frame" />
+    <origin xyz="0 0.1 0" rpy="-1.57 0 0" />
+  </joint>
+  <link name="usb_right_frame"/>
+  <joint name="usb_right_joint" type="fixed">
+      <parent link="base_link"/>
+      <child link="usb_right_frame"/>
+      <origin xyz="0 -0.1 0.0" rpy="1.57 3.14 0" />
+  </joint>
+  <link name="usb_front_frame"/>
+  <joint name="usb_front_joint" type="fixed">
+      <parent link="base_link"/>
+      <child link="usb_front_frame"/>
+      <origin xyz="0.1 0 0.0" rpy="-1.57 0 -1.57" />
+  </joint>
+  <link name="usb_back_frame"/>
+  <joint name="usb_back_joint" type="fixed">
+      <parent link="base_link"/>
+      <child link="usb_back_frame"/>
+      <origin xyz="-0.1 0 0.0" rpy="-1.57 0 1.57" />
+  </joint>
   <link name="livox_frame"> </link>
   <joint name="lidar_joint" type="fixed">
     <parent link="base_link" />
     <child link="livox_frame" />
-    <origin xyz="0 0 0.0" rpy="3.14 0.0 -1.57" />
+    <origin xyz="0.2 -0.1 0.0" rpy="3.14 0.0 -1.57" />
   </joint>
   <link name="imu_link"> </link>
